Commit message: update URDF to work better with viz

File: urdf/Arm_URDF_2025_live.urdf (robot description, URDF)
Before this commit: robot Arm_URDF_2025, 10 links, 9 joints
Links:
- added link real_camera_link, mass 0.0455289011770119; collision mesh filename=package://Arm_URDF_2025/meshes/camera_link.STL; visual mesh filename=package://Arm_URDF_2025/meshes/camera_link.STL
- added link real_finger_1, mass 0.131585801201098; collision mesh filename=package://Arm_URDF_2025/meshes/finger_1.STL; visual mesh filename=package://Arm_URDF_2025/meshes/finger_1.STL
- added link real_finger_2, mass 0.131585801201098; collision mesh filename=package://Arm_URDF_2025/meshes/finger_2.STL; visual mesh filename=package://Arm_URDF_2025/meshes/finger_2.STL
- added link real_link_1, mass 0.137634968166129; collision mesh filename=package://Arm_URDF_2025/meshes/link_1.STL; visual mesh filename=package://Arm_URDF_2025/meshes/link_1.STL
- added link real_link_2, mass 1.79663833155198; collision mesh filename=package://Arm_URDF_2025/meshes/link_2.STL; visual mesh filename=package://Arm_URDF_2025/meshes/link_2.STL
- added link real_link_3, mass 0.622999243464079; collision mesh filename=package://Arm_URDF_2025/meshes/link_3.STL; visual mesh filename=package://Arm_URDF_2025/meshes/link_3.STL
- added link real_link_4, mass 0.970122911594951; collision mesh filename=package://Arm_URDF_2025/meshes/link_4.STL; visual mesh filename=package://Arm_URDF_2025/meshes/link_4.STL
- added link real_link_5, mass 0.284717288401274; collision mesh filename=package://Arm_URDF_2025/meshes/link_5.STL; visual mesh filename=package://Arm_URDF_2025/meshes/link_5.STL
- added link real_link_6, mass 0.175170524925624; collision mesh filename=package://Arm_URDF_2025/meshes/link_6.STL; visual mesh filename=package://Arm_URDF_2025/meshes/link_6.STL
Joints:
- added joint real_camera_joint: type continuous, parent real_link_5, child real_camera_link, origin xyz=0.0756084691443581 0.0366419123913177 0.133665837449048 rpy=0 0 0, axis 0 1 0
- added joint real_finger_joint_1: type continuous, parent real_link_6, child real_finger_1, origin xyz=0.0342469999999999 0.0690450000000001 0.0150000000000005 rpy=0 0 0, axis 0 0 1
- added joint real_finger_joint_2: type continuous, parent real_link_6, child real_finger_2, origin xyz=0.0342469999999999 -0.0690460000000001 0.015 rpy=0 0 0, axis 0 0 -1
- added joint real_joint_1: type continuous, parent base_link, child real_link_1, origin xyz=0.06 0.06 0.0135 rpy=0 0 1.57, axis 0 0 -1
- added joint real_joint_2: type continuous, parent real_link_1, child real_link_2, origin xyz=1.24999999999858E-05 -0.03162775 0.0747000000000002 rpy=0 0 0, axis 0 -1 0
- added joint real_joint_3: type continuous, parent real_link_2, child real_link_3, origin xyz=-0.112992 0 0.384077 rpy=0 0 0, axis 0 1 0
- added joint real_joint_4: type continuous, parent real_link_3, child real_link_4, origin xyz=0.084452 0.036975 0.115 rpy=0 0 0, axis 1 0 0
- added joint real_joint_5: type continuous, parent real_link_4, child real_link_5, origin xyz=0.305479 -0.0406420000000001 0 rpy=0 0 0, axis 0 -1 0
- added joint real_joint_6: type continuous, parent real_link_5, child real_link_6, origin xyz=0.032 0.04064 0 rpy=0 0 0, axis 1 0 0
